File: Magnetometer_Breakout_IIS2MDCTR/Magnetometer_Breakout_IIS2MDCTR.kicad_pcb (KiCad board)
At the start: 2 copper layers, 16.5 x 19.7 mm, 6 parts, among them J1 Conn_01x07_Male, U1 IIS2MDCTR

Commit message: updated stuff seth said was bad
Routing:
- net GND: track 21.3 -> 3.72 mm, vias 0 -> 7
- net VDDIO: track 15.8 -> 17.4 mm
- net DRDY: track 8.96 -> 9.65 mm
- added copper zone on B.Cu, net GND
- added copper zone on F.Cu, net GND
Other:
- board size 16.5 x 19.7 mm -> 16.3 x 19.6 mm
- board text added: "CS"
- board text added: "DRDY"
- board text added: "GND"
- board text added: "SCL"
- board text added: "SDA"
- board text added: "VDD"
- board text added: "VDDIO"
- board text removed: "cs"
- board text removed: "drdy"
- board text removed: "gnd"
- board text removed: "scl"
- board text removed: "sda"
- board text removed: "vdd"
- board text removed: "vddio"
