File: MAGNETORQUERS/MAGNETORQUERS.kicad_pcb (KiCad board)
At the start: 2 copper layers, 32.4 x 22.8 mm, 13 parts, among them U1 DRV8876PWPR

Commit message: finalized board
 shrunk board size
relabeled pwm pin to reflect drv pin name
moved magnetorquer header pads closer
got rid of resistor/capacitor silkscreens, too small to see
edited drv8876 footprint to not have drc errors (increased via sizes, made thermal vias same pad #)
added more thermal vias on bottom cap directly below drv as recommended by datasheet
slightly adjusted copper fill areas in general to be cleaner
Parts:
- moved MAGN 5.76 mm to (139.6, 93.3)
- moved G*** 2.81 mm to (149.2, 78.2)
- moved 2.5kOhms 2.12 mm to (134.5, 89.8)
- renumbered 10kOhms to 10k, 16kOhms to 16k
Routing:
- net Earth: track 8.70 -> 3.68 mm, vias 6 -> 9
- net Net-(U1-VREF): track 18.9 -> 16.7 mm
- net Net-(STM1-Vcc): track 3.90 -> 5.92 mm
- net Net-(STM1-ADC): track 11.3 -> 9.74 mm
Other:
- board size 32.4 x 22.8 mm -> 32.4 x 20.2 mm
- board text added: "DRV8876PWPR"
- board text added: "EN/IN1"
- board text removed: "PWM"
