File: MAGNETORQUERS/MAGNETORQUERS.kicad_sch (KiCad schematic)
At the start: 12 parts, among them U1 DRV8876PWPR

Commit message: mag pwm control
Connections:
- net Earth: no longer U1.16 (PMODE)
- net at R1.2, REF_1.2, STM1.1 (Vcc): now also U1.16 (PMODE)
Changed lines of the file:
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@@
   (junction (at 78.74 68.58) (diameter 0) (color 0 0 0 0)
   )
+  (junction (at 44.45 139.7) (diameter 0) (color 0 0 0 0)
+  )
   (junction (at 148.59 74.93) (diameter 0) (color 0 0 0 0)
   )
@@
   (junction (at 85.09 107.95) (diameter 0) (color 0 0 0 0)
   )
-  (junction (at 129.54 147.32) (diameter 0) (color 0 0 0 0)
-  )
   (wire (pts (xy 149.86 106.68) (xy 158.75 106.68))
     (stroke (width 0) (type default))
@@
     (stroke (width 0) (type default))
   )
-  (wire (pts (xy 44.45 149.86) (xy 44.45 105.41))
+  (wire (pts (xy 44.45 149.86) (xy 44.45 139.7))
     (stroke (width 0) (type default))
   )
@@
     (stroke (width 0) (type default))
   )
+  (wire (pts (xy 44.45 139.7) (xy 44.45 105.41))
+    (stroke (width 0) (type default))
+  )
   (wire (pts (xy 167.64 74.93) (xy 167.64 55.88))
     (stroke (width 0) (type default))
@@
     (stroke (width 0) (type default))
   )
+  (wire (pts (xy 96.52 139.7) (xy 96.52 116.84))
+    (stroke (width 0) (type default))
+  )
   (wire (pts (xy 162.56 127) (xy 162.56 147.32))
     (stroke (width 0) (type default))
@@
     (stroke (width 0) (type default))
   )
-  (wire (pts (xy 96.52 116.84) (xy 96.52 143.51))
-    (stroke (width 0) (type default))
-  )
   (wire (pts (xy 80.01 149.86) (xy 87.63 149.86))
     (stroke (width 0) (type default))
@@
     (stroke (width 0) (type default))
   )
-  (wire (pts (xy 129.54 143.51) (xy 129.54 147.32))
-    (stroke (width 0) (type default))
-  )
   (wire (pts (xy 90.17 114.3) (xy 107.95 114.3))
     (stroke (width 0) (type default))
@@
     (stroke (width 0) (type default))
   )
+  (wire (pts (xy 44.45 139.7) (xy 96.52 139.7))
+    (stroke (width 0) (type default))
+  )
   (wire (pts (xy 90.17 68.58) (xy 105.41 68.58))
     (stroke (width 0) (type default))
@@
   )
   (wire (pts (xy 90.17 86.36) (xy 90.17 68.58))
-    (stroke (width 0) (type default))
-  )
-  (wire (pts (xy 96.52 143.51) (xy 129.54 143.51))
     (stroke (width 0) (type default))
   )
@@
       (effects (font (size 1.27 1.27)) hide)
     )
+    (pin "1")
+    (pin "2")
+    (pin "3")
+    (pin "4")
+    (pin "5")
     (pin "6")
     (pin "7")
-    (pin "5")
-    (pin "4")
-    (pin "3")
-    (pin "2")
-    (pin "1")
     (instances
       (project "MAGNETORQUERS"

Commit message: hi
Connections:
- net Earth renamed GND
